File: Sensors.kicad_sch (KiCad schematic)
At the start: 4 parts, among them U1 BME280

Commit message: Implement feature X to enhance user experience and fix bug Y in module Z
Parts:
- added C1: 10n, Capacitor_SMD:C_0805_2012Metric, symbol Device:C
- added C2, C3: 0.1u, Capacitor_SMD:C_0805_2012Metric, symbol Device:C
- added C4: 2.2u, Capacitor_SMD:C_0805_2012Metric, symbol Device:C
- added U2: MPU-6050, Sensor_Motion:InvenSense_QFN-24_4x4mm_P0.5mm, symbol Sensor_Motion:MPU-6050
Connections:
- net +3.3V: now also C1.1, C2.1, U2.13 (VDD), U2.8 (VLOGIC)
- net GND: now also C1.2, C2.2, C3.2, C4.2, U2.18 (GND)
- net I2C_SCL: now also U2.23 (SCL)
- net I2C_SDA: now also U2.24 (SDA)
- new net: C3.1, U2.10 (REGOUT)
- new net: C4.1, U2.20 (CPOUT)
- new net AUX_CL: U2.7 (AUX_CL)
- new net AUX_DA: U2.6 (AUX_DA)
- new net CLKIN: U2.1 (CLKIN)
- new net FSYNC: U2.11 (FSYNC)
- new net INT: U2.12 (INT)
- new net MPU_ADO: U2.9 (AD0)
Other:
- note added: "BME280 to measure temperatur,humidity and pressure MPU 6050 to determine the orientation and acceleration"
- note added: "MPU6050"
- company: (none) -> ODARI-DESIGNS
- title: (none) -> SENSORS

Commit message: Implement feature X to enhance user experience and fix bug Y in module Z
Parts:
- removed C1: 10n, Capacitor_SMD:C_0805_2012Metric, symbol Device:C
- removed C2, C3, C6: 0.1u, Capacitor_SMD:C_0805_2012Metric, symbol Device:C
- removed C4: 2.2u, Capacitor_SMD:C_0805_2012Metric, symbol Device:C
- removed R1, R2: 4.7K, Resistor_SMD:R_0603_1608Metric, symbol Device:R
- removed U1: BME280, Package_LGA:Bosch_LGA-8_2.5x2.5mm_P0.65mm_ClockwisePinNumbering, symbol Sensor:BME280
- removed U2: MPU-6050, Sensor_Motion:InvenSense_QFN-24_4x4mm_P0.5mm, symbol Sensor_Motion:MPU-6050
Other:
- note removed: "BME280 to measure temperatur,humidity and pressure MPU 6050 to determine the orientation and acceleration"
- note removed: "MPU6050"
- note removed: "PRESSURE SENSOR BME280"
- company: ODARI-DESIGNS -> (none)
- title: SENSORS -> (none)

Commit message: Implement feature X to enhance user experience and fix bug Y in module Z
Parts:
- added C6: 0.1u, Capacitor_SMD:C_0805_2012Metric, symbol Device:C
- added R1, R2: 4.7K, Resistor_SMD:R_0603_1608Metric, symbol Device:R
- added U1: BME280, Package_LGA:Bosch_LGA-8_2.5x2.5mm_P0.65mm_ClockwisePinNumbering, symbol Sensor:BME280
Connections:
- new net +3.3V: C6.1, R1.1, R2.1, U1.2 (CSB), U1.6 (VDDIO), U1.8 (VDD)
- new net GND: C6.2, U1.1 (GND), U1.5 (SDO), U1.7 (GND)
- new net I2C_SCL: R2.2, U1.4 (SCK)
- new net I2C_SDA: R1.2, U1.3 (SDI)
Other:
- note added: "PRESSURE SENSOR BME280"
