File: Sensors.kicad_sch (KiCad schematic)
At the start: 0 parts

Commit message: feat(sensors): define library symbols in schematic
Add standard library symbols for capacitors and resistors to the
Sensors schematic to enable component placement.
Parts:
- added C15, C16, C17, C18: 0.1u, Capacitor_SMD:C_0805_2012Metric, symbol Device:C
- added C19: 220p, Capacitor_SMD:C_0805_2012Metric, symbol Device:C
- added R20, R21, R22, R?: 4.7K, Resistor_SMD:R_0201_0603Metric, symbol Device:R
- added R23, R24: 47K5, Resistor_SMD:R_0201_0603Metric, symbol Device:R
- added U5: BME280, Package_LGA:Bosch_LGA-8_2.5x2.5mm_P0.65mm_ClockwisePinNumbering, symbol Sensor:BME280
- added U6: MPU-6050, Sensor_Motion:InvenSense_QFN-24_4x4mm_P0.5mm, symbol Sensor_Motion:MPU-6050
Connections:
- new net: R23.1, U6.6 (AUX_DA)
- new net: R24.1, U6.7 (AUX_CL)
- new net: C19.1, U6.20 (CPOUT)
- new net: C18.1, U6.10 (REGOUT)
- new net +3.3V: C15.1, C16.1, C17.1, R20.2, R21.1, R22.1, R23.2, R24.2, R?.2, U5.2 (CSB), U5.5 (SDO), U5.6 (VDDIO), U5.8 (VDD), U6.13 (VDD), U6.8 (VLOGIC)
- new net ADO: U6.9 (AD0)
- new net GND: C15.2, C16.2, C17.2, C18.2, C19.2, U5.1 (GND), U5.7 (GND), U6.1 (CLKIN), U6.11 (FSYNC), U6.18 (GND)
- new net INT: U6.12 (INT)
- new net SCL: R20.1, R22.2, U5.4 (SCK), U6.23 (SCL)
- new net SDA: R21.2, R?.1, U5.3 (SDI), U6.24 (SDA)
Other:
- note added: "BM280"
- note added: "MPU6050"
