File: iot_device_pcb.kicad_sch (KiCad schematic)
At the start: 25 parts, among them J1 USB_C_Receptacle_USB2.0_16P, J2 B2B-PH-K-S_LF__SN_, U2 AMS1117-3.3, U3 MCP73871

Commit message: feat(hw): update component references for consistency in PCB design
Parts:
- renumbered C3 to C1, C4 to C2, C1 to C3, C2 to C4, C6 to C5, J2 to J1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
