File: Display.kicad_sch (KiCad schematic)
At the start: 3 parts, among them J4 Conn_01x04_Pin, J5 Conn_01x04_Pin, J6 Conn_01x07_Pin

Commit message: refactor(sch): remove redundant GPIO labels
Remove multiple duplicate "GPIO" text labels from the schematic to clean up the drawing and prevent overlapping text elements.
Connections:
- net GPIO1: no longer J6.2 (Pin_2), J6.3 (Pin_3), J6.4 (Pin_4), J6.5 (Pin_5), J6.6 (Pin_6), J6.7 (Pin_7)
- new net GPIO2: J6.2 (Pin_2)
- new net GPIO3: J6.3 (Pin_3)
- new net GPIO4: J6.4 (Pin_4)
- new net GPIO5: J6.5 (Pin_5)
- new net GPIO6: J6.6 (Pin_6)
- new net GPIO7: J6.7 (Pin_7)
Changed lines of the file:
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@@
-		)
-	)
-	(label "GPIO"
-		(at 198.12 83.82 0)
-		(effects
-			(font
-				(size 1.27 1.27)
-			)
-			(justify left bottom)
-		)
-	)
-	(label "GPIO"
-		(at 198.12 86.36 0)
-		(effects
-			(font
-				(size 1.27 1.27)
-			)
-			(justify left bottom)
-		)
-	)
-	(label "GPIO"
-		(at 198.12 88.9 0)
-		(effects
-			(font
-				(size 1.27 1.27)
-			)
-			(justify left bottom)
 		)
 	)
@@
 				(thickness 0.254)
 				(bold yes)
-			)
-			(justify left bottom)
-		)
-	)
-	(label "GPIO"
-		(at 198.12 96.52 0)
-		(effects
-			(font
-				(size 1.27 1.27)
-			)
-			(justify left bottom)
-		)
-	)
-	(label "GPIO"
-		(at 198.12 91.44 0)
-		(effects
-			(font
-				(size 1.27 1.27)
 			)
 			(justify left bottom)
@@
 			)
 			(justify left bottom)
-		)
-	)
-	(label "GPIO"
-		(at 198.12 81.28 0)
-		(effects
-			(font
-				(size 1.27 1.27)
-			)
-			(justify left bottom)
-		)
-	)
-	(label "GPIO"
-		(at 198.12 93.98 0)
-		(effects
-			(font
-				(size 1.27 1.27)
-			)
-			(justify left bottom)
