File: Actuators.kicad_sch (KiCad schematic)
At the start: 0 parts

Commit message: feat(sch): add LTST-C170KRKT LED symbol to actuators schematic
Parts:
- added J3: Screw_Terminal_01x03, TerminalBlock_Phoenix:TerminalBlock_Phoenix_MKDS-1,5-3-5.08_1x03_P5.08mm_Horizontal, symbol Connector:Screw_Terminal_01x03
- added K1: RAYEX-L90, Relay_THT:Relay_1-Form-C_Schrack-RYII_RM3.2mm, symbol Relay:RAYEX-L90
- added LED7, LED8: LTST-C170KGKT, LED_SMD:LED_0805_2012Metric, symbol 2025-07-01_05-07-46:LTST-C170KRKT
- added Q3: BC817, Package_TO_SOT_SMD:SOT-23, symbol Transistor_BJT:BC817
- added R26, R27, R28: 470R, Resistor_SMD:R_0201_0603Metric, symbol Device:R
Connections:
- new net: J3.3 (Pin_3), K1.11A, K1.11B
- new net: J3.1 (Pin_1), K1.12
- new net: J3.2 (Pin_2), K1.14
- new net: K1.A1, Q3.2 (E), R27.2
- new net: Q3.1 (B), R28.1
- new net: LED8.2, R27.1
- new net: LED7.2, R26.1
- new net +3.3V: Q3.3 (C), R26.2
- new net FAN_RELAY: R28.2
- new net GND: K1.A2, LED7.1, LED8.1
Other:
- note added: "FAN_RELAY"
